File: Hardware/Schematics/ChipS.kicad_pcb (KiCad board)
At the start: 2 copper layers, 40 x 25 mm, 5 parts, among them J1 CONN_01X07, U1 PIC12C508

Commit message: Add files via upload
2nd hardware commit
Parts:
- removed GND: Measurement_Point_Round-TH_Small, Measurement_Points:Measurement_Point_Round-TH_Small
Routing:
- net /GP2: track 8.44 -> 9.03 mm
Other:
- net class Default: clearance 0.5 -> 0.4; trace_width 0.5 -> 0.8
- rule trace_clearance: 0.5 -> 0.4
- rule trace_min: 0.2 -> 0.5
- board text added: "07/2017"
- board text added: "T A P E"
- board text removed: "GND"
Changed lines of the file:
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@@
     (area 75.924999 58.924999 116.075001 84.075001)
     (thickness 1.6)
-    (drawings 27)
-    (tracks 20)
+    (drawings 37)
+    (tracks 21)
     (zones 0)
-    (modules 5)
+    (modules 4)
     (nets 10)
   )
@@
     (0 F.Cu signal)
     (31 B.Cu signal)
-    (32 B.Adhes user)
     (33 F.Adhes user)
-    (34 B.Paste user)
     (35 F.Paste user)
     (36 B.SilkS user)
@@
     (44 Edge.Cuts user)
     (45 Margin user)
-    (46 B.CrtYd user)
     (47 F.CrtYd user)
-    (48 B.Fab user)
     (49 F.Fab user)
   )
   (setup
-    (last_trace_width 0.5)
-    (trace_clearance 0.5)
+    (last_trace_width 0.8)
+    (trace_clearance 0.4)
     (zone_clearance 0.5)
     (zone_45_only no)
-    (trace_min 0.2)
+    (trace_min 0.5)
     (segment_width 0.2)
     (edge_width 0.15)
@@
     (visible_elements 7FFFFFFF)
     (pcbplotparams
-      (layerselection 0x00030_80000001)
-      (usegerberextensions false)
+      (layerselection 0x011f8_80000001)
+      (usegerberextensions true)
       (excludeedgelayer true)
       (linewidth 0.100000)
       (plotframeref false)
-      (viasonmask false)
+      (viasonmask true)
       (mode 1)
       (useauxorigin false)
@@
       (outputformat 1)
       (mirror false)
-      (drillshape 1)
+      (drillshape 0)
       (scaleselection 1)
-      (outputdirectory ""))
+      (outputdirectory Outputs/DrillDrawing/))
   )
   (net 0 "")
@@
   (net 9 /GP5)
   (net_class Default "Ceci est la Netclass par défaut"
-    (clearance 0.5)
-    (trace_width 0.5)
+    (clearance 0.4)
+    (trace_width 0.8)
     (via_dia 0.6)
     (via_drill 0.4)
@@
     (add_net VDD)
   )
-  (module Measurement_Points:Measurement_Point_Round-TH_Small (layer F.Cu)
-    (at 103.5 80)
-    (descr "Mesurement Point, Square, Trough Hole,  DM 1.5mm, Drill 0.8mm,")
-    (tags "Mesurement Point Round Trough Hole 1.5mm Drill 0.8mm")
-    (attr virtual)
-    (fp_text reference GND (at 3 0) (layer F.SilkS)
-      (effects (font (size 1 1) (thickness 0.15)))
-    )
-    (fp_text value Measurement_Point_Round-TH_Small (at 0 2) (layer F.Fab)
-      (effects (font (size 1 1) (thickness 0.15)))
-    )
-    (fp_circle (center 0 0) (end 1 0) (layer F.CrtYd) (width 0.05))
-    (pad 1 thru_hole circle (at 0 0) (size 1.5 1.5) (drill 0.8) (layers *.Cu *.Mask))
-  )
   (module Connectors_Molex:Molex_PicoBlade_53398-0771_07x1.25mm_Straight (layer F.Cu)
     (at 106.0609 69.7506 90)
@@
     (tags "connector molex picoblade smt")
     (attr smd)
-    (fp_text reference J1 (at -7.5 -2.575001 180) (layer F.SilkS)
+    (fp_text reference J1 (at -7.2494 -2.5609 180) (layer F.SilkS)
       (effects (font (size 1 1) (thickness 0.15)))
     )
@@
     )
   )
+  (gr_text 07/2017 (at 90 77) (layer B.SilkS)
+    (effects (font (size 1.5 1.5) (thickness 0.3)) (justify mirror))
+  )
+  (target plus (at 74 86) (size 5) (width 0.15) (layer Edge.Cuts))
+  (target plus (at 118 57) (size 5) (width 0.15) (layer Edge.Cuts))
+  (target plus (at 118 86) (size 5) (width 0.15) (layer Edge.Cuts))
+  (gr_text "T\n A\n  P\n   E" (at 111 68.5) (layer B.SilkS)
+    (effects (font (size 1.5 1.5) (thickness 0.3)) (justify mirror))
+  )
+  (gr_line (start 105 62) (end 112 62) (angle 90) (layer B.SilkS) (width 0.2))
+  (gr_line (start 105 75) (end 105 62) (angle 90) (layer B.SilkS) (width 0.2))
+  (gr_line (start 115 75) (end 105 75) (angle 90) (layer B.SilkS) (width 0.2))
+  (gr_line (start 115 62) (end 115 75) (angle 90) (layer B.SilkS) (width 0.2))
+  (gr_line (start 105 62) (end 115 62) (angle 90) (layer B.SilkS) (width 0.2))
+  (gr_text "T\nA\nP\nE" (at 79.5 71.5) (layer B.SilkS)
+    (effects (font (size 1.5 1.5) (thickness 0.3)) (justify mirror))
+  )
   (gr_line (start 77 81) (end 77 71) (angle 90) (layer B.SilkS) (width 0.2))
   (gr_line (start 82 81) (end 77 81) (angle 90) (layer B.SilkS) (width 0.2))
@@
   (gr_line (start 77 62) (end 82 62) (angle 90) (layer B.SilkS) (width 0.2))
   (gr_line (start 77 71) (end 77 62) (angle 90) (layer B.SilkS) (width 0.2))
-  (gr_text GND (at 96.5 61.5) (layer F.SilkS)
-    (effects (font (size 1 1) (thickness 0.2)) (justify left))
-  )
   (dimension 25 (width 0.3) (layer Dwgs.User)
     (gr_text "25,000 mm" (at 125.35 71.5 270) (layer Dwgs.User)
@@
     (effects (font (size 1.5 1.5) (thickness 0.3)))
   )
-  (gr_text 40x25 (at 111.75 61) (layer B.SilkS)
+  (gr_text 40x25 (at 88 80) (layer B.SilkS)
     (effects (font (size 1.5 1.5) (thickness 0.3)) (justify mirror))
   )
@@
   (gr_line (start 116 84) (end 76 84) (angle 90) (layer Edge.Cuts) (width 0.15))
   (gr_line (start 116 59) (end 116 84) (angle 90) (layer Edge.Cuts) (width 0.15))
-  (segment (start 94.796 72.3922) (end 94.796 70.542002) (width 0.5) (layer F.Cu) (net 3))
-  (segment (start 95.587402 69.7506) (end 104.6859 69.7506) (width 0.5) (layer F.Cu) (net 3))
-  (segment (start 94.796 70.542002) (end 95.587402 69.7506) (width 0.5) (layer F.Cu) (net 3))
-  (segment (start 97.336 72.3922) (end 97.336 71.5794) (width 0.5) (layer F.Cu) (net 4))
-  (segment (start 97.9148 71.0006) (end 104.6859 71.0006) (width 0.5) (layer F.Cu) (net 4))
-  (segment (start 97.336 71.5794) (end 97.9148 71.0006) (width 0.5) (layer F.Cu) (net 4))
-  (segment (start 80.5 66.5) (end 85.1 66.5) (width 0.5) (layer F.Cu) (net 5))
+  (segment (start 94.796 72.3922) (end 94.796 70.542002) (width 0.8) (layer F.Cu) (net 3))
+  (segment (start 94.796 70.542002) (end 95.587402 69.7506) (width 0.8) (layer F.Cu) (net 3))
+  (segment (start 95.587402 69.7506) (end 104.6859 69.7506) (width 0.8) (layer F.Cu) (net 3))
+  (segment (start 97.336 72.3922) (end 97.336 71.5794) (width 0.8) (layer F.Cu) (net 4))
+  (segment (start 97.336 71.5794) (end 97.9148 71.0006) (width 0.8) (layer F.Cu) (net 4))
+  (segment (start 97.9148 71.0006) (end 104.6859 71.0006) (width 0.8) (layer F.Cu) (net 4))
+  (segment (start 80.5 66.5) (end 85.1 66.5) (width 0.8) (layer F.Cu) (net 5))
+  (segment (start 97.336 64.7722) (end 97.336 65.3691) (width 0.8) (layer F.Cu) (net 6))
   (segment (start 97.336 64.7722) (end 97.336 65.3691) (width 0.5) (layer F.Cu) (net 6))
-  (segment (start 97.336 65.3691) (end 97.9675 66.0006) (width 0.5) (layer F.Cu) (net 6))
-  (segment (start 97.9675 66.0006) (end 104.6859 66.0006) (width 0.5) (layer F.Cu) (net 6))
+  (segment (start 97.336 65.3691) (end 97.9675 66.0006) (width 0.8) (layer F.Cu) (net 6))
+  (segment (start 97.9675 66.0006) (end 104.6859 66.0006) (width 0.8) (layer F.Cu) (net 6))
   (segment (start 97.336 64.7722) (end 97.336 65.0008) (width 0.5) (layer F.Cu) (net 6))
-  (segment (start 94.796 64.7722) (end 94.796 66.2962) (width 0.5) (layer F.Cu) (net 7))
-  (segment (start 95.7504 67.2506) (end 104.6859 67.2506) (width 0.5) (layer F.Cu) (net 7))
-  (segment (start 94.796 66.2962) (end 95.7504 67.2506) (width 0.5) (layer F.Cu) (net 7))
-  (segment (start 104.6859 68.5006) (end 93.7365 68.5006) (width 0.5) (layer F.Cu) (net 8))
-  (segment (start 92.256 67.0201) (end 92.256 64.7722) (width 0.5) (layer F.Cu) (net 8))
-  (segment (start 93.7365 68.5006) (end 92.256 67.0201) (width 0.5) (layer F.Cu) (net 8))
-  (segment (start 85.1 70.5) (end 91.583 70.5) (width 0.5) (layer F.Cu) (net 9))
-  (segment (start 92.256 71.173) (end 92.256 72.3922) (width 0.5) (layer F.Cu) (net 9))
-  (segment (start 91.583 70.5) (end 92.256 71.173) (width 0.5) (layer F.Cu) (net 9))
+  (segment (start 94.796 64.7722) (end 94.796 66.2962) (width 0.8) (layer F.Cu) (net 7))
+  (segment (start 94.796 66.2962) (end 95.7504 67.2506) (width 0.8) (layer F.Cu) (net 7))
+  (segment (start 95.7504 67.2506) (end 104.6859 67.2506) (width 0.8) (layer F.Cu) (net 7))
+  (segment (start 104.6859 68.5006) (end 93.7365 68.5006) (width 0.8) (layer F.Cu) (net 8))
+  (segment (start 93.7365 68.5006) (end 92.256 67.0201) (width 0.8) (layer F.Cu) (net 8))
+  (segment (start 92.256 67.0201) (end 92.256 64.7722) (width 0.8) (layer F.Cu) (net 8))
+  (segment (start 85.1 70.5) (end 91.583 70.5) (width 0.8) (layer F.Cu) (net 9))
+  (segment (start 91.583 70.5) (end 92.256 71.173) (width 0.8) (layer F.Cu) (net 9))
+  (segment (start 92.256 71.173) (end 92.256 72.3922) (width 0.8) (layer F.Cu) (net 9))
   (zone (net 0) (net_name "") (layer F.SilkS) (hatch edge 0.508)
-    (connect_pads yes (clearance 0.5))
+    (connect_pads (clearance 0.5))
     (min_thickness 0.25)
     (fill yes (arc_segments 16) (thermal_gap 0.5) (thermal_bridge_width 0.5))
@@
   (zone (net 1) (net_name VDD) (layer F.Cu) (hatch edge 0.508)
     (priority 1)
-    (connect_pads yes (clearance 0.5))
+    (connect_pads (clearance 0.5))
     (min_thickness 0.25)
     (fill yes (arc_segments 16) (thermal_gap 0.5) (thermal_bridge_width 0.5))
@@
   )
   (zone (net 2) (net_name GND) (layer F.Cu) (hatch edge 0.508)
-    (connect_pads yes (clearance 0.5))
+    (connect_pads (clearance 0.5))
     (min_thickness 0.25)
     (fill yes (arc_segments 16) (thermal_gap 0.5) (thermal_bridge_width 0.5))
@@
   (zone (net 0) (net_name "") (layer B.SilkS) (hatch edge 0.508)
     (priority 1)
-    (connect_pads yes (clearance 0.5))
+    (connect_pads (clearance 0.5))
     (min_thickness 0.25)
     (fill yes (arc_segments 16) (thermal_gap 0.5) (thermal_bridge_width 0.5))
@@
     )
   )
-  (zone (net 0) (net_name "") (layer F.Mask) (hatch edge 0.508)
-    (priority 1)
-    (connect_pads yes (clearance 0.5))
+  (zone (net 2) (net_name GND) (layer B.Cu) (hatch edge 0.508)
+    (connect_pads (clearance 0.5))
     (min_thickness 0.25)
     (fill yes (arc_segments 16) (thermal_gap 0.5) (thermal_bridge_width 0.5))
-    (polygon
-      (pts
-        (xy 102.5 63.5) (xy 100 63.5) (xy 100 61) (xy 102.5 61)
-      )
-    )
-  )
-  (zone (net 2) (net_name GND) (layer B.Cu) (hatch edge 0.508)
-    (connect_pads yes (clearance 0.5))
-    (min_thickness 0.25)
-    (fill yes (arc_segments 16) (thermal_gap 0.5) (thermal_bridge_width 0.5))
