File: Hardware/Schematics/ChipS.sch (KiCad schematic (older format))
At the start: 4 parts, among them J1 CONN_01X07, U1 PIC12C508

Commit message: Add files via upload
2nd hardware commit
Parts:
- added J2: CONN_01X07, symbol CONN_01X07
Connections:
- wire segments 30 -> 37
Other:
- note added: "Cable"
- note added: "PCB Schematic"
- note added: "Power-Supply\n"
- note added: "Signals"
- note added: "To ChipS Board"
- note added: "To PSX Main Board"
- moved on the sheet: D1, J1, R1, U1
